File: 50x70_tiny.kicad_pcb (KiCad board)
At the start: 2 copper layers, 78.2 x 78.5 mm, 20 parts, among them J1 Barrel_Jack_MountingPin, J2 Conn_01x04_F, J3 Conn_02x03_M, Q1 Q_NMOS_GDS, SW1 SW_MEC_5E, SW2 SW_MEC_5E, U1 ATtiny85, U2 L78L05_TO92

Commit message: redesign, 3D models and a picture
Parts:
- added ?: , , F.Cu at (149.5, 103.7)
- added R8: 10kΩ, Resistor_THT:R_Axial_DIN0207_L6.3mm_D2.5mm_P7.62mm_Horizontal, F.Cu at (152.1, 84.0)
- added SW3: SW_MEC_5E, Button_Switch_THT:SW_PUSH_6mm_H4.3mm, F.Cu at (154.8, 90.5)
- J2: footprint Connector_PinHeader_2.54mm:PinHeader_1x04_P2.54mm_Vertical -> Connector_PinSocket_2.54mm:PinSocket_1x04_P2.54mm_Vertical
- J3: footprint Connector_PinSocket_2.54mm:PinSocket_2x03_P2.54mm_Vertical -> Connector_PinHeader_2.54mm:PinHeader_2x03_P2.54mm_Vertical
- moved R2 7.55 mm to (162.7, 89.2), turned to 0 degrees
- moved C2 7.25 mm to (144.8, 87.2), turned to -90 degrees
- moved U2 6.53 mm to (139.5, 84.5), turned to -90 degrees
- moved R6 5.80 mm to (162.5, 86.1)
- moved R4 5.58 mm to (165.8, 78.4)
- moved R3 5.46 mm to (169.0, 86.1)
- moved J3 2.57 mm to (178.0, 73.2)
- moved C1 1.46 mm to (135.8, 86.0)
- moved SW1 1.03 mm to (180.2, 84.0)
- moved SW2 1.00 mm to (180.2, 91.5)
- moved TH1 1.00 mm to (148.3, 91.5)
Routing:
- net GND: track 15.4 -> 2.69 mm
- net Net-(R2-Pad1): track 20.9 -> 29.5 mm
- net +5V: track 84.1 -> 91.8 mm
- net Net-(J3-Pad6): track 30.7 -> 35.9 mm
- net Net-(R3-Pad2): track 16.9 -> 15.0 mm
- net Net-(R4-Pad2): track 20.6 -> 18.9 mm
- net VCC: track 2100.8 -> 2099.5 mm
- net Net-(D1-Pad2): track 73.3 -> 72.7 mm
- net Net-(J2-Pad2): track 46.4 -> 45.9 mm
Other:
- outline, holes or cut-outs redrawn
- board text added: "70x50mm TinyReflow V1,2 CC-BY 4,0"
- board text added: "RESET"
- board text removed: "70x50mm TinyReflow V1,1 CC-BY 4,0"

Commit message: mix
Other:
- board text added: "70x50mm TinyReflow V1,2 CERN-OHL-P v2"
- board text removed: "70x50mm TinyReflow V1,2 CC-BY 4,0"
Changed lines of the file:
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@@
     (pad "2" thru_hole oval (at 2.54 0) (size 1.4 1.4) (drill 0.7) (layers *.Cu *.Mask)
       (net 9 "Net-(R2-Pad1)") (pintype "passive"))
-    (model "${KICAD6_3DMODEL_DIR}/Resistor_THT.3dshapes/R_Axial_DIN0204_L3.6mm_D1.6mm_P2.54mm_Vertical.wrl"
-      (offset (xyz 0 0 0))
+    (model "${KIPRJMOD}/weirdthermistor.stp"
+      (offset (xyz 0 0 -2.25))
       (scale (xyz 1 1 1))
-      (rotate (xyz 0 0 0))
+      (rotate (xyz 0 0 90))
     )
   )
@@
     (effects (font (size 1.5 1.5) (thickness 0.3)))
   )
-  (gr_text "70x50mm TinyReflow V1,2 CC-BY 4,0" (at 108.5 119.25 270) (layer "F.SilkS")
-    (effects (font (size 1.5 1.5) (thickness 0.375)))
+  (gr_text "70x50mm TinyReflow V1,2 CERN-OHL-P v2" (at 108.5 119.5 270) (layer "F.SilkS")
+    (effects (font (size 1.3 1.3) (thickness 0.3)))
   )
   (segment (start 135.75 86) (end 136.75 86) (width 0.75) (layer "F.Cu") (net 1))

Commit message: gerber and stuff
Other:
- board text added: "JLCJLCJLCJLC"
Changed lines of the file:
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@@
     (effects (font (size 1.5 1.5) (thickness 0.3)))
+  )
+  (gr_text "JLCJLCJLCJLC" (at 183.35 84.4 90) (layer "F.SilkS")
+    (effects (font (size 1 1) (thickness 0.16)))
   )
   (gr_text "70x50mm TinyReflow V1,2 CERN-OHL-P v2" (at 108.5 119.5 270) (layer "F.SilkS")

Commit message: bom+
Parts:
- Q1: value Q_NMOS_GDS -> 30N06
- TH1: value 10kΩ -> 10kΩ bead thermistor
Other:
- board text removed: "JLCJLCJLCJLC"
Changed lines of the file:
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@@
       (effects (font (size 1 1) (thickness 0.15)))
     )
-    (fp_text value "10kΩ" (at 1.27 1.92) (layer "F.Fab")
+    (fp_text value "10kΩ bead thermistor" (at 1.27 1.92) (layer "F.Fab")
       (effects (font (size 1 1) (thickness 0.15)))
     )
@@
       (effects (font (size 1 1) (thickness 0.15)))
     )
-    (fp_text value "Q_NMOS_GDS" (at 2.54 2.9025) (layer "F.Fab")
+    (fp_text value "30N06" (at 2.54 2.9025) (layer "F.Fab")
       (effects (font (size 1 1) (thickness 0.15)))
     )
@@
     (effects (font (size 1.5 1.5) (thickness 0.3)))
   )
-  (gr_text "JLCJLCJLCJLC" (at 183.35 84.4 90) (layer "F.SilkS")
-    (effects (font (size 1 1) (thickness 0.16)))
-  )
   (gr_text "70x50mm TinyReflow V1,2 CERN-OHL-P v2" (at 108.5 119.5 270) (layer "F.SilkS")
