File: 50x70_tiny.kicad_sch (KiCad schematic)
At the start: 20 parts, among them J1 Barrel_Jack_MountingPin, J2 Conn_01x04_F, J3 Conn_02x03_M, Q1 Q_NMOS_GDS, SW1 SW_MEC_5E, SW2 SW_MEC_5E, U1 ATtiny85, U2 L78L05_TO92

Commit message: redesign, 3D models and a picture
Parts:
- added R8: 10kΩ, Resistor_THT:R_Axial_DIN0207_L6.3mm_D2.5mm_P7.62mm_Horizontal, symbol Device:R_Small
- added SW3: SW_MEC_5E, Button_Switch_THT:SW_PUSH_6mm_H4.3mm, symbol Switch:SW_MEC_5E
- J2: footprint Connector_PinHeader_2.54mm:PinHeader_1x04_P2.54mm_Vertical -> Connector_PinSocket_2.54mm:PinSocket_1x04_P2.54mm_Vertical
- J3: footprint Connector_PinSocket_2.54mm:PinSocket_2x03_P2.54mm_Vertical -> Connector_PinHeader_2.54mm:PinHeader_2x03_P2.54mm_Vertical
Connections:
- net +5V: now also R8.2
- net GND: now also SW3.2
- net at J3.6 (Pin_6), U1.1 (~{RESET}/PB5): now also R8.1, SW3.1
Changed lines of the file:
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@@
   (junction (at 189.23 115.57) (diameter 0) (color 0 0 0 0)
   )
+  (junction (at 187.96 82.55) (diameter 0) (color 0 0 0 0)
+  )
   (junction (at 151.13 33.02) (diameter 0) (color 0 0 0 0)
   )
@@
   (junction (at 85.09 64.77) (diameter 0) (color 0 0 0 0)
   )
+  (junction (at 187.96 71.12) (diameter 0) (color 0 0 0 0)
+  )
   (junction (at 167.64 57.15) (diameter 0) (color 0 0 0 0)
   )
@@
     (stroke (width 0) (type default) (color 0 0 0 0))
   )
+  (wire (pts (xy 205.74 85.09) (xy 205.74 87.63))
+    (stroke (width 0) (type default) (color 0 0 0 0))
+  )
   (wire (pts (xy 124.46 80.01) (xy 124.46 82.55))
     (stroke (width 0) (type default) (color 0 0 0 0))
@@
     (stroke (width 0) (type default) (color 0 0 0 0))
   )
+  (wire (pts (xy 184.15 74.93) (xy 184.15 77.47))
+    (stroke (width 0) (type default) (color 0 0 0 0))
+  )
   (wire (pts (xy 177.8 29.21) (xy 185.42 29.21))
     (stroke (width 0) (type default) (color 0 0 0 0))
@@
     (stroke (width 0) (type default) (color 0 0 0 0))
   )
+  (wire (pts (xy 187.96 71.12) (xy 187.96 82.55))
+    (stroke (width 0) (type default) (color 0 0 0 0))
+  )
   (wire (pts (xy 189.23 93.98) (xy 189.23 95.25))
     (stroke (width 0) (type default) (color 0 0 0 0))
@@
     (stroke (width 0) (type default) (color 0 0 0 0))
   )
+  (wire (pts (xy 201.93 85.09) (xy 205.74 85.09))
+    (stroke (width 0) (type default) (color 0 0 0 0))
+  )
   (wire (pts (xy 170.18 57.15) (xy 167.64 57.15))
     (stroke (width 0) (type default) (color 0 0 0 0))
@@
     (stroke (width 0) (type default) (color 0 0 0 0))
   )
+  (wire (pts (xy 184.15 82.55) (xy 187.96 82.55))
+    (stroke (width 0) (type default) (color 0 0 0 0))
+  )
   (wire (pts (xy 82.55 59.69) (xy 85.09 59.69))
     (stroke (width 0) (type default) (color 0 0 0 0))
@@
   )
   (wire (pts (xy 166.37 102.87) (xy 171.45 102.87))
+    (stroke (width 0) (type default) (color 0 0 0 0))
+  )
+  (wire (pts (xy 187.96 82.55) (xy 191.77 82.55))
     (stroke (width 0) (type default) (color 0 0 0 0))
   )
@@
     )
     (pin "1")
+    (pin "2")
+  )
+  (symbol (lib_id "Switch:SW_MEC_5E") (at 196.85 85.09 0) (unit 1)
+    (in_bom yes) (on_board yes) (fields_autoplaced)
+    (property "Reference" "SW3" (id 0) (at 196.85 74.93 0))
+    (property "Value" "SW_MEC_5E" (id 1) (at 196.85 77.47 0))
+    (property "Footprint" "Button_Switch_THT:SW_PUSH_6mm_H4.3mm" (id 2) (at 196.85 77.47 0)
+      (effects (font (size 1.27 1.27)) hide)
+    )
+    (property "Datasheet" "http://www.apem.com/int/index.php?controller=attachment&id_attachment=1371" (id 3) (at 196.85 77.47 0)
+      (effects (font (size 1.27 1.27)) hide)
+    )
+    (pin "1")
+    (pin "1")
+    (pin "2")
     (pin "2")
   )
@@
     (property "Reference" "J3" (id 0) (at 198.12 59.69 0))
     (property "Value" "Conn_02x03_M" (id 1) (at 198.12 62.23 0))
-    (property "Footprint" "Connector_PinSocket_2.54mm:PinSocket_2x03_P2.54mm_Vertical" (id 2) (at 196.85 73.66 0)
+    (property "Footprint" "Connector_PinHeader_2.54mm:PinHeader_2x03_P2.54mm_Vertical" (id 2) (at 196.85 73.66 0)
       (effects (font (size 1.27 1.27)) hide)
     )
@@
       (effects (font (size 1.27 1.27)) (justify left))
     )
-    (property "Footprint" "Connector_PinHeader_2.54mm:PinHeader_1x04_P2.54mm_Vertical" (id 2) (at 166.37 73.66 0)
+    (property "Footprint" "Connector_PinSocket_2.54mm:PinSocket_1x04_P2.54mm_Vertical" (id 2) (at 166.37 73.66 0)
       (effects (font (size 1.27 1.27)) hide)
     )
@@
     (pin "2")
   )
+  (symbol (lib_id "power:+5V") (at 184.15 74.93 0) (unit 1)
+    (in_bom yes) (on_board yes)
+    (property "Reference" "#PWR0122" (id 0) (at 184.15 78.74 0)
+      (effects (font (size 1.27 1.27)) hide)
+    )
+    (property "Value" "+5V" (id 1) (at 184.15 71.12 0))
+    (property "Footprint" "" (id 2) (at 184.15 74.93 0)
+      (effects (font (size 1.27 1.27)) hide)
+    )
+    (property "Datasheet" "" (id 3) (at 184.15 74.93 0)
+      (effects (font (size 1.27 1.27)) hide)
+    )
+    (pin "1")
+  )
   (symbol (lib_id "power:+5V") (at 208.28 62.23 0) (unit 1)
     (in_bom yes) (on_board yes)
@@
     (pin "2")
   )
+  (symbol (lib_id "Device:R_Small") (at 184.15 80.01 180) (unit 1)
+    (in_bom yes) (on_board yes)
+    (property "Reference" "R8" (id 0) (at 181.61 81.2801 0)
+      (effects (font (size 1.27 1.27)) (justify left))
+    )
+    (property "Value" "10kΩ" (id 1) (at 181.61 78.7401 0)
+      (effects (font (size 1.27 1.27)) (justify left))
+    )
+    (property "Footprint" "Resistor_THT:R_Axial_DIN0207_L6.3mm_D2.5mm_P7.62mm_Horizontal" (id 2) (at 184.15 80.01 0)
+      (effects (font (size 1.27 1.27)) hide)
+    )
+    (property "Datasheet" "~" (id 3) (at 184.15 80.01 0)
+      (effects (font (size 1.27 1.27)) hide)
+    )
+    (pin "1")
+    (pin "2")
+  )
   (symbol (lib_id "power:VCC") (at 142.24 22.86 0) (unit 1)
     (in_bom yes) (on_board yes) (fields_autoplaced)
@@
     (pin "1")
     (pin "2")
+  )
+  (symbol (lib_id "power:GND") (at 205.74 87.63 0) (unit 1)
+    (in_bom yes) (on_board yes) (fields_autoplaced)
+    (property "Reference" "#PWR0121" (id 0) (at 205.74 93.98 0)
+      (effects (font (size 1.27 1.27)) hide)
+    )
+    (property "Value" "GND" (id 1) (at 205.74 92.71 0))
+    (property "Footprint" "" (id 2) (at 205.74 87.63 0)
+      (effects (font (size 1.27 1.27)) hide)
+    )
+    (property "Datasheet" "" (id 3) (at 205.74 87.63 0)
+      (effects (font (size 1.27 1.27)) hide)
+    )
+    (pin "1")
   )
   (symbol (lib_id "power:GND") (at 143.51 113.03 0) (unit 1)
@@
       (reference "#PWR0120") (unit 1) (value "GND") (footprint "")
     )
+    (path "/f1bbc9a0-1a8c-486c-92a2-f4acda30268f"
+      (reference "#PWR0121") (unit 1) (value "GND") (footprint "")
+    )
+    (path "/c9951c49-864c-42d1-97d3-23d57e53f9f7"
+      (reference "#PWR0122") (unit 1) (value "+5V") (footprint "")
+    )
     (path "/927d37d4-8eae-4b4f-a0f2-f5a1f882477c"
       (reference "C1") (unit 1) (value "330nf") (footprint "Capacitor_THT:C_Disc_D5.0mm_W2.5mm_P2.50mm")
@@
     )
     (path "/b697066c-54ff-4ee3-b116-388c7a0e739e"
-      (reference "J2") (unit 1) (value "Conn_01x04_F") (footprint "Connector_PinHeader_2.54mm:PinHeader_1x04_P2.54mm_Vertical")
+      (reference "J2") (unit 1) (value "Conn_01x04_F") (footprint "Connector_PinSocket_2.54mm:PinSocket_1x04_P2.54mm_Vertical")
     )
     (path "/958bb47a-472d-4af5-9706-e1f8d5630753"
-      (reference "J3") (unit 1) (value "Conn_02x03_M") (footprint "Connector_PinSocket_2.54mm:PinSocket_2x03_P2.54mm_Vertical")
+      (reference "J3") (unit 1) (value "Conn_02x03_M") (footprint "Connector_PinHeader_2.54mm:PinHeader_2x03_P2.54mm_Vertical")
     )
     (path "/e4eab4cc-19dc-499c-ac8b-0e005ff66c2f"
@@
       (reference "R7") (unit 1) (value "10kΩ") (footprint "Resistor_THT:R_Axial_DIN0207_L6.3mm_D2.5mm_P7.62mm_Horizontal")
     )
+    (path "/d8609345-02c0-4326-adab-d5f0d551dcbe"
+      (reference "R8") (unit 1) (value "10kΩ") (footprint "Resistor_THT:R_Axial_DIN0207_L6.3mm_D2.5mm_P7.62mm_Horizontal")
+    )
     (path "/c305b044-7927-4e38-8daf-dc4f915fef90"
       (reference "SW1") (unit 1) (value "SW_MEC_5E") (footprint "Button_Switch_THT:SW_PUSH_6mm_H4.3mm")
@@
       (reference "SW2") (unit 1) (value "SW_MEC_5E") (footprint "Button_Switch_THT:SW_PUSH_6mm_H4.3mm")
     )
+    (path "/1ceb027d-8905-4c6c-9b1c-e0a5a8ae4681"
+      (reference "SW3") (unit 1) (value "SW_MEC_5E") (footprint "Button_Switch_THT:SW_PUSH_6mm_H4.3mm")
+    )
     (path "/e69511c1-f354-4934-9e4a-94ceeec46854"

Commit message: bom+
Parts:
- Q1: value Q_NMOS_GDS -> 30N06
- TH1: value 10kΩ -> 10kΩ bead thermistor
Connections:
- net at SW3.1: now also J3.6 (Pin_6), R8.1, U1.1 (~{RESET}/PB5)
Changed lines of the file:
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@@
       (effects (font (size 1.27 1.27)) (justify left))
     )
-    (property "Value" "Q_NMOS_GDS" (id 1) (at 181.61 58.4199 0)
+    (property "Value" "30N06" (id 1) (at 181.61 58.4199 0)
       (effects (font (size 1.27 1.27)) (justify left))
     )
@@
       (effects (font (size 1.27 1.27)) (justify left))
     )
-    (property "Value" "10kΩ" (id 1) (at 149.86 82.55 0)
+    (property "Value" "10kΩ bead thermistor" (id 1) (at 149.86 82.55 0)
       (effects (font (size 1.27 1.27)) (justify left))
     )
@@
     )
     (path "/e4eab4cc-19dc-499c-ac8b-0e005ff66c2f"
-      (reference "Q1") (unit 1) (value "Q_NMOS_GDS") (footprint "Package_TO_SOT_THT:TO-220F-3_Vertical")
+      (reference "Q1") (unit 1) (value "30N06") (footprint "Package_TO_SOT_THT:TO-220F-3_Vertical")
     )
     (path "/0f10a37a-0e05-4c1f-a806-953bbb6e5e8b"
@@
     )
     (path "/e69511c1-f354-4934-9e4a-94ceeec46854"
-      (reference "TH1") (unit 1) (value "10kΩ") (footprint "Resistor_THT:R_Axial_DIN0204_L3.6mm_D1.6mm_P2.54mm_Vertical")
+      (reference "TH1") (unit 1) (value "10kΩ bead thermistor") (footprint "Resistor_THT:R_Axial_DIN0204_L3.6mm_D1.6mm_P2.54mm_Vertical")
     )
     (path "/3d7b53e5-dcb4-4b1e-983c-0426e9c51da4"
